File: LM2597-Fixed/LM2597-Fixed.kicad_sch (KiCad schematic)
At the start: 9 parts, among them IC1 LM2597MX-5.0_NOPB, J1 Conn_01x05

Commit message: routed and drc'ed
Parts:
- removed C1, C2: 0.1uF, Capacitor_THT:C_Disc_D4.7mm_W2.5mm_P5.00mm, symbol Device:C
- removed J1: Conn_01x05, Connector_PinHeader_2.54mm:PinHeader_1x05_P2.54mm_Vertical, symbol Connector_Generic:Conn_01x05
- added C3 (x2): 0.1uF, Capacitor_SMD:C_0603_1608Metric_Pad1.08x0.95mm_HandSolder, symbol Device:C
- added J1: Conn_01x03, Connector_PinHeader_2.54mm:PinHeader_1x03_P2.54mm_Vertical, symbol Connector_Generic:Conn_01x03
Connections:
- net +VDC: now also J1.1 (Pin_1)
- net GND: now also C3.2, C3.2, J1.3 (Pin_3)
- net at IC1.2 (DELAY): now also C3.1
- net at IC1.5 (~{SHUTDOWN}/SOFT-START): now also C3.1
- net +5V renamed VCC
- net VCC: now also J1.2 (Pin_2)

Commit message: updated all of these to SMD parts
Parts:
- C3: footprint Capacitor_SMD:C_0603_1608Metric_Pad1.08x0.95mm_HandSolder -> Capacitor_SMD:C_1206_3216Metric_Pad1.33x1.80mm_HandSolder
- R1: footprint Resistor_THT:R_Axial_DIN0207_L6.3mm_D2.5mm_P5.08mm_Vertical -> Resistor_SMD:R_1206_3216Metric_Pad1.30x1.75mm_HandSolder
